File: rpi_pmod_hub/rpi_pmod_hub.kicad_pcb (KiCad board)
At the start: 2 copper layers, 0 parts

Commit message: WIP 20220907
Parts:
- added C1: 100nF, Capacitor_SMD:C_0603_1608Metric, F.Cu at (169.4, 102.0)
- added C2: 100nF, Capacitor_SMD:C_0603_1608Metric, F.Cu at (169.4, 79.0)
- added J1: PMOD_U, Connector_PinHeader_2.54mm:PinHeader_2x06_P2.54mm_Horizontal, F.Cu at (158.3, 89.7)
- added J2: PMOD_L, Connector_PinHeader_2.54mm:PinHeader_2x06_P2.54mm_Horizontal, F.Cu at (158.3, 112.5)
- added J3: RPI_EXT_SMD, Connector_PinHeader_2.54mm:PinHeader_2x20_P2.54mm_Vertical_SMD, B.Cu at (176.2, 122.1)
- added J4: HUB75, Connector_PinHeader_2.54mm:PinHeader_2x08_P2.54mm_Vertical_SMD, F.Cu at (174.9, 94.6)
- added JP1: SET DIR, Jumper:SolderJumper-3_P1.3mm_Bridged12_RoundedPad1.0x1.5mm_NumberLabels, F.Cu at (157.0, 93.5)
- added JP2: SET EN, Jumper:SolderJumper-3_P1.3mm_Bridged12_RoundedPad1.0x1.5mm_NumberLabels, F.Cu at (157.0, 96.0)
- added RN1: R_Pack04, Resistor_SMD:R_Array_Convex_4x0402, F.Cu at (161.7, 107.6)
- added RN2: R_Pack04, Resistor_SMD:R_Array_Convex_4x0402, F.Cu at (161.7, 84.7)
- added RN3: R_Pack04, Resistor_SMD:R_Array_Convex_4x0402, F.Cu at (161.7, 105.0)
- added RN4: R_Pack04, Resistor_SMD:R_Array_Convex_4x0402, F.Cu at (161.7, 82.0)
- added RN5: R_Pack04, Resistor_SMD:R_Array_Convex_4x0402, F.Cu at (172.5, 108.3)
- added RN6: R_Pack04, Resistor_SMD:R_Array_Convex_4x0402, F.Cu at (172.5, 82.6)
- added RN7: R_Pack04, Resistor_SMD:R_Array_Convex_4x0402, F.Cu at (172.5, 105.6)
- added RN8: R_Pack04, Resistor_SMD:R_Array_Convex_4x0402, F.Cu at (172.5, 85.3)
- added U1: 74HC245, Package_SO:TSSOP-20_4.4x6.5mm_P0.65mm, F.Cu at (167.1, 106.3)
- added U2: 74HC245, Package_SO:TSSOP-20_4.4x6.5mm_P0.65mm, F.Cu at (167.1, 83.3)
Routing:
- net +3V3: track 0.00 -> 119.6 mm, vias 0 -> 5
- net /IO_L18_T2_34+: track 0.00 -> 84.6 mm
- net /IO_L15_T2_DQS_AD12_35+: track 0.00 -> 77.1 mm, vias 0 -> 2
- net /IO_L18_T2_34-: track 0.00 -> 76.6 mm, vias 0 -> 4
- net /IO_L15_T2_DQS_AD12_35-: track 0.00 -> 75.8 mm, vias 0 -> 2
- net /IO_L11_T1_SRCC_13+: track 0.00 -> 70.2 mm
- net /IO_L11_T1_SRCC_13-: track 0.00 -> 69.1 mm
- net /IO_L13_T2_MRCC_13+: track 0.00 -> 58.4 mm
- net /IO_L15_T2_DQS_13+: track 0.00 -> 55.4 mm, vias 0 -> 2
- net /IO_L17_T2_34+: track 0.00 -> 55.4 mm
- net /IO_L13_T2_MRCC_13-: track 0.00 -> 54.8 mm, vias 0 -> 2
- net /IO_L15_T2_DQS_13-: track 0.00 -> 54.6 mm, vias 0 -> 2
- net GND: track 0.00 -> 44.5 mm, vias 0 -> 2
- net /IO_L14_T2_SRCC_13+: track 0.00 -> 40.4 mm
- net /XCVR_EN: track 0.00 -> 40.3 mm, vias 0 -> 3
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Other:
- board outline added: 51.8 x 51.4 mm
- board text added: "5"
