File: rpi_pmod_hub/rpi_pmod_hub.kicad_sch (KiCad schematic)
At the start: 4 parts

Commit message: WIP 20220907
Parts:
- added C1, C2: 100nF, Capacitor_SMD:C_0603_1608Metric, symbol Device:C
- added J4: HUB75, Connector_PinHeader_2.54mm:PinHeader_2x08_P2.54mm_Vertical_SMD, symbol Connector_Generic:Conn_02x08_Odd_Even
- added JP1: SET DIR, Jumper:SolderJumper-3_P1.3mm_Bridged12_RoundedPad1.0x1.5mm_NumberLabels, symbol Jumper:SolderJumper_3_Bridged12
- added JP2: SET EN, Jumper:SolderJumper-3_P1.3mm_Bridged12_RoundedPad1.0x1.5mm_NumberLabels, symbol Jumper:SolderJumper_3_Bridged12
- added RN1, RN2, RN3, RN4, RN5, RN6, RN7, RN8: R_Pack04, Resistor_SMD:R_Array_Convex_4x0402, symbol Device:R_Pack04
- added U2: 74HC245, Package_SO:TSSOP-20_4.4x6.5mm_P0.65mm, symbol 74xx:74HC245
- J1, J2: renamed from J?; footprint (none) -> Connector_PinHeader_2.54mm:PinHeader_2x06_P2.54mm_Horizontal; symbol Connector_Generic:Conn_02x06_Top_Bottom -> Connector_Generic:Conn_02x06_Odd_Even
- J3: renamed from J?; footprint (none) -> Connector_PinHeader_2.54mm:PinHeader_2x20_P2.54mm_Vertical_SMD
- U1: renamed from U?; footprint (none) -> Package_SO:TSSOP-20_4.4x6.5mm_P0.65mm
Connections:
- net IO_L13N_T2_MRCC_13 is gone; now on net GND: J1.4 (Pin_4), J3.10 (Pin_10)
- net IO_L15N_T2_DQS_13 is gone; now on net GND: J2.4 (Pin_4), J3.33 (Pin_33)
- net IO_L15P_T2_DQS_13 is gone; now on net GND: J2.3 (Pin_3), J3.19 (Pin_19)
- net IO_L21N_T3_DQS_13 is gone; now on net IO_L15_T2_DQS_AD12_35-: J3.21 (Pin_21)
- net +3V3: now also J1.1 (Pin_1), J1.2 (Pin_2), J2.1 (Pin_1), J2.2 (Pin_2), J3.18 (Pin_18), J3.2 (Pin_2), U1.20 (VCC), C1.1, C2.1, JP1.1 (A), JP2.1 (A), U2.20 (VCC); no longer J1.12 (Pin_12), J1.6 (Pin_6), J2.12 (Pin_12), J2.6 (Pin_6), J3.1 (Pin_1), J3.17 (Pin_17)
- net +5V: now also J3.1 (Pin_1), J3.3 (Pin_3); no longer J3.2 (Pin_2), J3.4 (Pin_4)
- net GND: now also J1.3 (Pin_3), J3.13 (Pin_13), J3.26 (Pin_26), J3.29 (Pin_29), J3.40 (Pin_40), J3.5 (Pin_5), U1.10 (GND), C1.2, C2.2, JP1.3 (B), JP2.3 (B), U2.10 (GND); no longer J1.11 (Pin_11), J1.5 (Pin_5), J2.11 (Pin_11), J2.5 (Pin_5), J3.14 (Pin_14), J3.20 (Pin_20), J3.25 (Pin_25), J3.30 (Pin_30), J3.34 (Pin_34), J3.39 (Pin_39), J3.6 (Pin_6), J3.9 (Pin_9)
- net RPIO_0: now also J3.28 (Pin_28); no longer J3.27 (Pin_27)
- net RPIO_1: now also J3.27 (Pin_27); no longer J3.28 (Pin_28)
- net RPIO_2: now also J3.4 (Pin_4); no longer J3.3 (Pin_3)
- net RPIO_3: now also J3.6 (Pin_6); no longer J3.5 (Pin_5)
- net RPIO_4: now also J3.8 (Pin_8); no longer J3.7 (Pin_7)
- net RPIO_5: now also J3.30 (Pin_30); no longer J3.29 (Pin_29)
- net RPIO_6: now also J3.32 (Pin_32); no longer J3.31 (Pin_31)
- net RPIO_7: now also J3.25 (Pin_25); no longer J3.26 (Pin_26)
- net XCVR_DIR: now reaches U1.1 (A->B)
- net XCVR_DIR: now also JP1.2 (C), U2.1 (A->B)
- net at U1.11 (B7): now also RN5.8 (R1.2)
- net at U1.12 (B6): now also RN5.7 (R2.2)
- net at U1.13 (B5): now also RN5.6 (R3.2)
- net at U1.14 (B4): now also RN5.5 (R4.2)
- net at U1.15 (B3): now also RN7.8 (R1.2)
- net at U1.16 (B2): now also RN7.7 (R2.2)
- net at U1.17 (B1): now also RN7.6 (R3.2)
- net at U1.18 (B0): now also RN7.5 (R4.2)
- net XCVR_EN: now reaches U1.19 (CE)
- net XCVR_EN: now also JP2.2 (C), U2.19 (CE)
- net at U1.2 (A0): now also RN3.8 (R1.2)
- net at U1.3 (A1): now also RN3.7 (R2.2)
- net at U1.4 (A2): now also RN3.6 (R3.2)
- net at U1.5 (A3): now also RN3.5 (R4.2)
- net at U1.6 (A4): now also RN1.8 (R1.2)
- net at U1.7 (A5): now also RN1.7 (R2.2)
- net at U1.8 (A6): now also RN1.6 (R3.2)
- net at U1.9 (A7): now also RN1.5 (R4.2)
- removed net IO_L11N_T1_SRCC_13: J2.2 (Pin_2), J3.13 (Pin_13)
- net IO_L11P_T1_SRCC_13 renamed IO_L17_T2_34+
- net IO_L17_T2_34+: now also J2.11 (Pin_11), RN3.1 (R1.1); no longer J2.1 (Pin_1)
- removed net IO_L13P_T2_MRCC_13: J1.3 (Pin_3), J3.18 (Pin_18)
- net IO_L14N_T2_SRCC_13 renamed IO_L12_T1_MRCC_34+
- net IO_L12_T1_MRCC_34+: now also J2.8 (Pin_8), RN1.2 (R2.1); no longer J2.10 (Pin_10)
- net IO_L14P_T2_SRCC_13 renamed IO_L17_T2_34-
- net IO_L17_T2_34-: now also J3.31 (Pin_31), RN3.3 (R3.1); no longer J3.40 (Pin_40)
- net IO_L15N_T2_DQS_AD12N_35 renamed IO_L15_T2_DQS_AD12_35-
- net IO_L15_T2_DQS_AD12_35-: now also RN4.4 (R4.1); no longer J3.22 (Pin_22)
- net IO_L15P_T2_DQS_AD12P_35 renamed IO_L11_T1_SRCC_13-
- net IO_L11_T1_SRCC_13-: now also J3.14 (Pin_14), RN4.3 (R3.1); no longer J3.24 (Pin_24)
- net IO_L16N_T2_13 renamed IO_L12_T1_MRCC_34-
- net IO_L12_T1_MRCC_34-: now also J2.6 (Pin_6), RN1.4 (R4.1)
- net IO_L16P_T2_13 renamed IO_L15_T2_DQS_AD12_35+
- net IO_L15_T2_DQS_AD12_35+: now also J1.12 (Pin_12), RN4.2 (R2.1)
- net IO_L17N_T2_13 renamed IO_L18_T2_34-
- net IO_L18_T2_34-: now also J1.6 (Pin_6), RN2.4 (R4.1)
- removed net IO_L1N_T0_AD0N_35: J1.2 (Pin_2), J3.32 (Pin_32)
- net IO_L1P_T0_AD0P_35 renamed IO_L11_T1_SRCC_13+
- net IO_L11_T1_SRCC_13+: now also J1.11 (Pin_11), RN4.1 (R1.1); no longer J1.1 (Pin_1)
- net IO_L22N_T3_13 renamed IO_L17_T2_13-
- net IO_L17_T2_13-: no longer J2.8 (Pin_8)
- net IO_L22P_T3_13 renamed IO_L13_T2_MRCC_13+
- net IO_L13_T2_MRCC_13+: now also J3.17 (Pin_17), RN1.1 (R1.1); no longer J3.8 (Pin_8)
- net IO_L2N_T0_AD8P_35 renamed IO_L16_T2_13-
- net IO_L16_T2_13-: no longer J1.8 (Pin_8)
- net IO_L2P_T0_AD8P_35 renamed IO_L14_T2_SRCC_13-
- net IO_L14_T2_SRCC_13-: now also J2.10 (Pin_10), RN3.4 (R4.1); no longer J1.7 (Pin_7)
- new net: J4.1 (Pin_1), RN6.8 (R1.2)
- new net: J4.10 (Pin_10), RN7.1 (R1.1)
- new net: J4.11 (Pin_11), RN8.7 (R2.2)
- new net: J4.12 (Pin_12), RN7.2 (R2.1)
- new net: J4.13 (Pin_13), RN8.6 (R3.2)
- new net: J4.14 (Pin_14), RN7.3 (R3.1)
- new net: J4.15 (Pin_15), RN8.5 (R4.2)
- new net: J4.16 (Pin_16), RN7.4 (R4.1)
- new net: J4.2 (Pin_2), RN5.1 (R1.1)
- new net: J4.3 (Pin_3), RN6.7 (R2.2)
- new net: J4.4 (Pin_4), RN5.2 (R2.1)
- new net: J4.5 (Pin_5), RN6.6 (R3.2)
- new net: J4.6 (Pin_6), RN5.3 (R3.1)
- new net: J4.7 (Pin_7), RN6.5 (R4.2)
- new net: J4.8 (Pin_8), RN5.4 (R4.1)
- new net: J4.9 (Pin_9), RN8.8 (R1.2)
- new net: RN6.1 (R1.1), U2.18 (B0)
- new net: RN6.2 (R2.1), U2.17 (B1)
- new net: RN6.3 (R3.1), U2.16 (B2)
- new net: RN6.4 (R4.1), U2.15 (B3)
- new net: RN8.1 (R1.1), U2.14 (B4)
- new net: RN8.2 (R2.1), U2.13 (B5)
- new net: RN8.3 (R3.1), U2.12 (B6)
- new net: RN8.4 (R4.1), U2.11 (B7)
- new net: RN4.8 (R1.2), U2.2 (A0)
- new net: RN4.7 (R2.2), U2.3 (A1)
- new net: RN4.6 (R3.2), U2.4 (A2)
- new net: RN4.5 (R4.2), U2.5 (A3)
- new net: RN2.8 (R1.2), U2.6 (A4)
- new net: RN2.7 (R2.2), U2.7 (A5)
- new net: RN2.6 (R3.2), U2.8 (A6)
- new net: RN2.5 (R4.2), U2.9 (A7)
- new net IO_L13_T2_MRCC_13-: J2.5 (Pin_5), J3.9 (Pin_9), RN1.3 (R3.1)
- new net IO_L14_T2_SRCC_13+: J2.12 (Pin_12), J3.39 (Pin_39), RN3.2 (R2.1)
- new net IO_L15_T2_DQS_13+: J1.7 (Pin_7), J3.20 (Pin_20), RN2.1 (R1.1)
- new net IO_L15_T2_DQS_13-: J1.5 (Pin_5), J3.34 (Pin_34), RN2.3 (R3.1)
- new net IO_L16_T2_13+: J3.24 (Pin_24)
- new net IO_L18_T2_34+: J1.8 (Pin_8), J3.7 (Pin_7), RN2.2 (R2.1)
- new net IO_L21_T3_DQS_13-: J3.22 (Pin_22)
- no-connect marks 10 -> 8
Other:
- note added: "<- PYNQ NORTH"
- moved on the sheet: J1, J2, U1
